File: docs/stickpointv-ch32v003-v1.0.0-semantics.kicad_sch (KiCad schematic)
At the start: 9 parts, among them U1 joystick-b10k, U2 CH32V003J4M6

Commit message: update document
Other:
- company: (none) -> 74th
- title: (none) -> StickPointV
Changed lines of the file:
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@@
 (kicad_sch (version 20230121) (generator eeschema)
   (paper "A4")
+  (title_block
+    (title "StickPointV")
+    (date "2024-01-06")
+    (rev "1.0.0")
+    (company "74th")
+  )
   (junction (at 95.25 123.19) (diameter 0) (color 0 0 0 0)
   )
